File: kicad/speaker.kicad_sch (KiCad schematic)
At the start: 5 parts, among them J9 PC Speaker, Q4 2N5225

Commit message: update kicad project
Parts:
- C113: seq_coord (none) -> L30
- J9: seq_coord (none) -> L33
- Q4: seq_coord (none) -> L31
- R40: seq_coord (none) -> L32; seq_silkscreen R40 -> (none)
- R41: seq_coord (none) -> M31
Changed lines of the file:
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@@
 			)
 		)
-		(property "seq_coord" ""
+		(property "seq_coord" "L32"
 			(at 91.44 67.31 0)
 			(effects
@@
 			)
 		)
-		(property "seq_silkscreen" "R40"
+		(property "seq_silkscreen" ""
 			(at 91.44 67.31 0)
 			(effects
@@
 		)
 		(property "seq_notes" "Green,Black,Black,Gold"
+			(at 91.44 67.31 0)
+			(effects
+				(font
+					(size 1.27 1.27)
+				)
+				(hide yes)
+			)
+		)
+		(property "seq_port" ""
 			(at 91.44 67.31 0)
 			(effects
@@
 			)
 		)
-		(property "seq_coord" ""
+		(property "seq_coord" "L33"
 			(at 144.78 57.15 0)
 			(effects
@@
 			)
 		)
-		(property "seq_coord" ""
+		(property "seq_coord" "L30"
 			(at 118.11 67.31 0)
 			(effects
@@
 			)
 		)
-		(property "seq_coord" ""
+		(property "seq_coord" "L31"
 			(at 101.6 67.31 0)
 			(effects
@@
 			)
 		)
-		(property "seq_coord" ""
+		(property "seq_coord" "M31"
 			(at 129.54 57.15 0)
 			(effects
