File: kicad/lightpen.kicad_sch (KiCad schematic)
At the start: 4 parts, among them J16 Light Pen, U141 74LS74, U89 74LS04

Commit message: update kicad project
Parts:
- J16, R69: seq_coord (none) -> M1
- U141: seq_coord (none) -> I15; seq_silkscreen (none) -> LS74
- U89: seq_coord (none) -> L11; seq_silkscreen (none) -> LS04
Changed lines of the file:
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@@
+	(wire
+		(pts
+			(xy 97.79 78.74) (xy 97.79 128.27)
+		)
+		(stroke
+			(width 0)
+			(type default)
+		)
+	)
 	(wire
 		(pts
@@
 	(wire
 		(pts
-			(xy 97.79 78.74) (xy 97.79 100.33)
-		)
-		(stroke
-			(width 0)
-			(type default)
-		)
-	)
-	(wire
-		(pts
 			(xy 185.42 73.66) (xy 185.42 85.09)
 		)
@@
 	(wire
 		(pts
-			(xy 142.24 86.36) (xy 144.78 86.36)
+			(xy 142.24 86.36) (xy 152.4 86.36)
 		)
 		(stroke
@@
 	(hierarchical_label "~{LP_STB}"
 		(shape input)
-		(at 144.78 86.36 0)
+		(at 152.4 86.36 0)
 		(effects
 			(font
@@
 			)
 		)
-		(property "seq_coord" ""
+		(property "seq_coord" "M1"
 			(at 104.14 78.74 0)
 			(effects
@@
 			)
 		)
-		(property "seq_coord" ""
+		(property "seq_coord" "M1"
 			(at 86.36 81.28 0)
 			(effects
@@
 	(symbol
 		(lib_id "power:GND")
-		(at 97.79 100.33 0)
+		(at 97.79 128.27 0)
 		(unit 1)
 		(exclude_from_sim no)
@@
 		(fields_autoplaced yes)
 		(property "Reference" "#PWR042"
-			(at 97.79 106.68 0)
+			(at 97.79 134.62 0)
 			(effects
 				(font
@@
 		)
 		(property "Value" "GND"
-			(at 97.79 105.41 0)
+			(at 97.79 133.35 0)
 			(effects
 				(font
@@
 		)
 		(property "Footprint" ""
-			(at 97.79 100.33 0)
+			(at 97.79 128.27 0)
 			(effects
 				(font
@@
 		)
 		(property "Datasheet" ""
-			(at 97.79 100.33 0)
+			(at 97.79 128.27 0)
 			(effects
 				(font
@@
 		)
 		(property "Description" "Power symbol creates a global label with name \"GND\" , ground"
-			(at 97.79 100.33 0)
+			(at 97.79 128.27 0)
 			(effects
 				(font
@@
 			)
 		)
-		(property "seq_coord" ""
+		(property "seq_coord" "L11"
 			(at 130.81 86.36 0)
 			(effects
@@
 			)
 		)
-		(property "seq_silkscreen" ""
+		(property "seq_silkscreen" "LS04"
 			(at 130.81 86.36 0)
 			(effects
@@
 			)
 		)
-		(property "seq_coord" ""
+		(property "seq_coord" "I15"
 			(at 185.42 92.71 0)
 			(effects
@@
 			)
 		)
-		(property "seq_silkscreen" ""
+		(property "seq_silkscreen" "LS74"
 			(at 185.42 92.71 0)
 			(effects

Commit message: More updates
Parts:
- R69: value ??Ω -> 4.7kΩ; seq_notes (none) -> Yellow, Violet, Red, Gold
Connections:
- no-connect marks 0 -> 1
Other:
- note added: "To 6845"
- title: (none) -> Video Unit: Light Pen Header
- moved on the sheet: R69, U89B
