File: kicad/composite_video.kicad_sch (KiCad schematic)
At the start: 1 part, among them J10 Composite Jack

Commit message: update kicad project
Parts:
- J10: seq_coord (none) -> J33
Other:
- moved on the sheet: J10
Changed lines of the file:
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@@
 	(wire
 		(pts
-			(xy 140.97 78.74) (xy 170.18 78.74)
+			(xy 116.84 87.63) (xy 146.05 87.63)
 		)
 		(stroke
@@
 	(wire
 		(pts
-			(xy 165.1 76.2) (xy 165.1 88.9)
+			(xy 140.97 85.09) (xy 140.97 97.79)
 		)
 		(stroke
@@
 	(wire
 		(pts
-			(xy 165.1 76.2) (xy 170.18 76.2)
+			(xy 140.97 85.09) (xy 146.05 85.09)
 		)
 		(stroke
@@
 	)
 	(label "COMPOSITE_OUT"
-		(at 140.97 78.74 0)
+		(at 116.84 87.63 0)
 		(effects
 			(font
@@
 	(symbol
 		(lib_id "Connector_Generic:Conn_01x02")
-		(at 175.26 76.2 0)
+		(at 151.13 85.09 0)
 		(unit 1)
 		(exclude_from_sim no)
@@
 		(dnp no)
 		(property "Reference" "J10"
-			(at 177.8 76.1999 0)
+			(at 153.67 85.0899 0)
 			(effects
 				(font
@@
 		)
 		(property "Value" "Composite Jack"
-			(at 177.8 78.7399 0)
+			(at 153.67 87.6299 0)
 			(effects
 				(font
@@
 		)
 		(property "Footprint" "Connector_PinHeader_2.54mm:PinHeader_1x02_P2.54mm_Horizontal"
-			(at 175.26 76.2 0)
+			(at 151.13 85.09 0)
 			(effects
 				(font
@@
 		)
 		(property "Datasheet" "~"
-			(at 175.26 76.2 0)
+			(at 151.13 85.09 0)
 			(effects
 				(font
@@
 		)
 		(property "Description" "Generic connector, single row, 01x02, script generated (kicad-library-utils/schlib/autogen/connector/)"
-			(at 175.26 76.2 0)
+			(at 151.13 85.09 0)
 			(effects
 				(font
@@
 		)
 		(property "seq_partno" ""
-			(at 175.26 76.2 0)
+			(at 151.13 85.09 0)
 			(effects
 				(font
@@
 			)
 		)
-		(property "seq_coord" ""
-			(at 175.26 76.2 0)
+		(property "seq_coord" "J33"
+			(at 151.13 85.09 0)
 			(effects
 				(font
@@
 		)
 		(property "seq_silkscreen" ""
-			(at 175.26 76.2 0)
+			(at 151.13 85.09 0)
 			(effects
 				(font
@@
 		)
 		(property "seq_sharpie" ""
-			(at 175.26 76.2 0)
+			(at 151.13 85.09 0)
 			(effects
 				(font
@@
 		)
 		(property "seq_notes" ""
-			(at 175.26 76.2 0)
+			(at 151.13 85.09 0)
 			(effects
 				(font
@@
 	(symbol
 		(lib_id "power:GND")
-		(at 165.1 88.9 0)
+		(at 140.97 97.79 0)
 		(unit 1)
 		(exclude_from_sim no)
@@
 		(fields_autoplaced yes)
 		(property "Reference" "#PWR075"
-			(at 165.1 95.25 0)
+			(at 140.97 104.14 0)
 			(effects
 				(font
@@
 		)
 		(property "Value" "GND"
-			(at 165.1 93.98 0)
+			(at 140.97 102.87 0)
 			(effects
 				(font
@@
 		)
 		(property "Footprint" ""
-			(at 165.1 88.9 0)
+			(at 140.97 97.79 0)
 			(effects
 				(font
@@
 		)
 		(property "Datasheet" ""
-			(at 165.1 88.9 0)
+			(at 140.97 97.79 0)
 			(effects
 				(font
@@
 		)
 		(property "Description" "Power symbol creates a global label with name \"GND\" , ground"
-			(at 165.1 88.9 0)
+			(at 140.97 97.79 0)
 			(effects
 				(font

Commit message: More updates
Parts:
- added U131: 74LS240, Package_DIP:DIP-20_W7.62mm, symbol 74xx:74LS240
- added U132, U133: 74LS74, Package_DIP:DIP-14_W7.62mm, symbol 74xx:74LS74
- added U139: 74LS86, Package_DIP:DIP-14_W7.62mm, symbol 74xx:74LS86
- added U151: PAL20L2, Package_DIP:DIP-24_W7.62mm, symbol seequa:PAL20L2
Connections:
- net GND: now also U131.1 (OEa), U131.10 (GND), U151.12 (GND), U151.13 (I_{13})
- new net: U139.4, U151.19 (~{O_{2}})
- new net: U132.1 (~{R}), U132.4 (~{S}), U133.1 (~{R}), U133.10 (~{S}), U133.13 (~{R}), U133.4 (~{S}), U139.3
- new net: U131.4 (I1a), U151.18 (~{O_{1}})
- new net +5V: U131.20 (VCC), U139.1, U139.5, U151.24 (V_{CC})
- new net 14MHz: U133.11 (C)
- new net BLUE_{CLK}: U132.6 (~{Q}), U151.6 (I_{5})
- new net BW: U139.2, U151.22 (I_{19})
- new net C0_{BODGE_IN}: U151.1 (I_{0})
- new net CLT_{O2}: U131.2 (I0a), U139.6
- new net CMP_{b}: U151.21 (I_{18})
- new net CMP_{g}: U151.20 (I_{17})
- new net CMP_{r}: U151.17 (I_{16})
- new net CRTC_HS: U151.3 (I_{2})
- new net CRTC_VS: U151.4 (I_{3})
- new net CYAN_{CLK}: U133.6 (~{Q}), U151.8 (I_{7})
- new net FRONT_PORCH: U151.23 (I_{12})
- new net GRAPHICS: U151.2 (I_{1})
- new net GREEN_{CLK}: U133.8 (~{Q}), U151.16 (I_{15})
- new net HSYNC_{SERR}: U131.17 (I3b)
- new net MAGENTA_{CLK}: U133.9 (Q), U151.15 (I_{14})
- new net RED_{CLK}: U133.12 (D), U133.5 (Q), U151.9 (I_{8})
- new net VMEM_{EN}: U151.5 (I_{4})
- new net VSYNC_OUT: U139.12
- new net YELLOW_{CLK}: U132.5 (Q), U133.2 (D), U151.7 (I_{6})
- new net ~{14MHz}: U132.3 (C), U133.3 (C)
- new net ~{3.58MHz}: U132.2 (D)
- new net ~{HSYNC_{SERR}}: U139.11
- new net ~{HSYNC}: U139.13
- no-connect marks 0 -> 2
Other:
- title: (none) -> Video Unit: Composite Generation
- moved on the sheet: J10

Commit message: Add parallel port, game port
Connections:
- net HSYNC_{SERR} is gone; now on net ~{HSYNC_{SERR}}: U131.17 (I3b)
- net CMP_{b}: now also U131.6 (I2a)
- net CMP_{g}: now also U131.13 (I1b)
- net CMP_{r}: now also U131.8 (I3a)
- net GND: now also U131.19 (OEb)
- net ~{HSYNC}: no longer U139.13
- net CMP_{I}: now reaches U131.15 (I2b)
- new net HSYNC: U139.13
Changed lines of the file:
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@@
+	)
+	(junction
+		(at 232.41 83.82)
+		(diameter 0)
+		(color 0 0 0 0)
 	)
 	(junction
@@
 	(wire
 		(pts
+			(xy 218.44 71.12) (xy 236.22 71.12)
+		)
+		(stroke
+			(width 0)
+			(type default)
+		)
+	)
+	(wire
+		(pts
 			(xy 232.41 91.44) (xy 248.92 91.44)
 		)
@@
 	(wire
 		(pts
-			(xy 232.41 81.28) (xy 232.41 91.44)
+			(xy 232.41 81.28) (xy 232.41 83.82)
+		)
+		(stroke
+			(width 0)
+			(type default)
+		)
+	)
+	(wire
+		(pts
+			(xy 218.44 63.5) (xy 236.22 63.5)
 		)
 		(stroke
@@
 	(wire
 		(pts
-			(xy 71.12 90.17) (xy 80.01 90.17)
+			(xy 46.99 90.17) (xy 80.01 90.17)
+		)
+		(stroke
+			(width 0)
+			(type default)
+		)
+	)
+	(wire
+		(pts
+			(xy 217.17 73.66) (xy 236.22 73.66)
 		)
 		(stroke
@@
 	(wire
 		(pts
+			(xy 232.41 83.82) (xy 232.41 91.44)
+		)
+		(stroke
+			(width 0)
+			(type default)
+		)
+	)
+	(wire
+		(pts
 			(xy 154.94 17.78) (xy 200.66 17.78)
 		)
@@
 	(wire
 		(pts
+			(xy 232.41 83.82) (xy 236.22 83.82)
+		)
+		(stroke
+			(width 0)
+			(type default)
+		)
+	)
+	(wire
+		(pts
 			(xy 46.99 118.11) (xy 55.88 118.11)
 		)
@@
 	(wire
 		(pts
-			(xy 133.35 66.04) (xy 144.78 66.04)
+			(xy 129.54 66.04) (xy 144.78 66.04)
 		)
 		(stroke
@@
 	(wire
 		(pts
-			(xy 133.35 63.5) (xy 144.78 63.5)
+			(xy 129.54 63.5) (xy 144.78 63.5)
 		)
 		(stroke
@@
 	(wire
 		(pts
-			(xy 133.35 60.96) (xy 144.78 60.96)
+			(xy 129.54 60.96) (xy 144.78 60.96)
 		)
 		(stroke
@@
 	(wire
 		(pts
-			(xy 133.35 58.42) (xy 144.78 58.42)
+			(xy 129.54 58.42) (xy 144.78 58.42)
 		)
 		(stroke
@@
 			(width 0)
 			(type default)
+		)
+	)
+	(label "CMP_{i}"
+		(at 218.44 73.66 0)
+		(effects
+			(font
+				(size 1.27 1.27)
+			)
+			(justify left bottom)
 		)
 	)
@@
 		)
 	)
+	(label "CMP_{r}"
+		(at 218.44 66.04 0)
+		(effects
+			(font
+				(size 1.27 1.27)
+			)
+			(justify left bottom)
+		)
+	)
 	(label "RED_{CLK}"
 		(at 114.3 59.69 180)
@@
 		)
 	)
-	(label "CRTC_HS"
-		(at 133.35 60.96 0)
-		(effects
-			(font
-				(size 1.27 1.27)
-			)
-			(justify left bottom)
-		)
-	)
 	(label "~{HSYNC_{SERR}}"
 		(at 87.63 120.65 180)
@@
 		)
 	)
+	(label "BW"
+		(at 35.56 36.83 180)
+		(effects
+			(font
+				(size 1.27 1.27)
+			)
+			(justify right bottom)
+		)
+	)
 	(label "MAGENTA_{CLK}"
 		(at 179.07 55.88 180)
@@
 		)
 	)
-	(label "GRAPHICS"
-		(at 133.35 58.42 0)
+	(label "CMP_{g}"
+		(at 218.44 71.12 0)
 		(effects
 			(font
@@
 		)
 	)
-	(label "VMEM_{EN}"
-		(at 133.35 66.04 0)
-		(effects
-			(font
-				(size 1.27 1.27)
-			)
-			(justify left bottom)
+	(label "CMP_{r}"
+		(at 179.07 60.96 180)
+		(effects
+			(font
+				(size 1.27 1.27)
+			)
+			(justify right bottom)
 		)
 	)
@@
 		)
 	)
+	(label "CMP_{b}"
+		(at 218.44 63.5 0)
+		(effects
+			(font
+				(size 1.27 1.27)
+			)
+			(justify left bottom)
+		)
+	)
+	(label "CMP_{g}"
+		(at 179.07 63.5 180)
+		(effects
+			(font
+				(size 1.27 1.27)
+			)
+			(justify right bottom)
+		)
+	)
 	(label "BW"
 		(at 179.07 68.58 180)
@@
 		)
 	)
-	(label "HSYNC_{SERR}"
+	(label "CMP_{b}"
+		(at 179.07 66.04 180)
+		(effects
+			(font
+				(size 1.27 1.27)
+			)
+			(justify right bottom)
+		)
+	)
+	(label "~{HSYNC_{SERR}}"
 		(at 222.25 76.2 0)
 		(effects
@@
 			)
 			(justify right bottom)
-		)
-	)
-	(label "CRTC_VS"
-		(at 133.35 63.5 0)
-		(effects
-			(font
-				(size 1.27 1.27)
-			)
-			(justify left bottom)
 		)
 	)
@@
 		)
 	)
+	(hierarchical_label "HSYNC"
+		(shape input)
+		(at 46.99 123.19 180)
+		(effects
+			(font
+				(size 1.27 1.27)
+			)
+			(justify right)
+		)
+	)
 	(hierarchical_label "C0_{BODGE_IN}"
 		(shape input)
@@
 		)
 	)
+	(hierarchical_label "CMP_{I}"
+		(shape input)
+		(at 217.17 73.66 180)
+		(effects
+			(font
+				(size 1.27 1.27)
+			)
+			(justify right)
+		)
+	)
+	(hierarchical_label "CRTC_VS"
+		(shape input)
+		(at 129.54 63.5 180)
+		(effects
+			(font
+				(size 1.27 1.27)
+			)
+			(justify right)
+		)
+	)
 	(hierarchical_label "~{3.58MHz}"
 		(shape input)
@@
 		)
 	)
+	(hierarchical_label "CRTC_HS"
+		(shape input)
+		(at 129.54 60.96 180)
+		(effects
+			(font
+				(size 1.27 1.27)
+			)
+			(justify right)
+		)
+	)
+	(hierarchical_label "VSYNC_OUT"
+		(shape input)
+		(at 46.99 118.11 180)
+		(effects
+			(font
+				(size 1.27 1.27)
+			)
+			(justify right)
+		)
+	)
+	(hierarchical_label "VMEM_{EN}"
+		(shape input)
+		(at 129.54 66.04 180)
+		(effects
+			(font
+				(size 1.27 1.27)
+			)
+			(justify right)
+		)
+	)
 	(hierarchical_label "~{HSYNC}"
 		(shape input)
-		(at 46.99 123.19 180)
+		(at 46.99 128.27 180)
 		(effects
 			(font
@@
 		)
 	)
-	(hierarchical_label "VSYNC_OUT"
-		(shape input)
-		(at 46.99 118.11 180)
+	(hierarchical_label "CMP_{g}"
+		(shape input)
+		(at 180.34 63.5 0)
+		(effects
+			(font
+				(size 1.27 1.27)
+			)
+			(justify left)
+		)
+	)
+	(hierarchical_label "GRAPHICS"
+		(shape input)
+		(at 129.54 58.42 180)
 		(effects
 			(font
@@
 		)
 	)
-	(hierarchical_label "CMP_{g}"
-		(shape input)
-		(at 180.34 63.5 0)
+	(hierarchical_label "BW"
+		(shape input)
+		(at 29.21 36.83 180)
+		(effects
+			(font
+				(size 1.27 1.27)
+			)
+			(justify right)
+		)
+	)
+	(hierarchical_label "~{14MHz}"
+		(shape input)
+		(at 71.12 34.29 180)
+		(effects
+			(font
+				(size 1.27 1.27)
+			)
+			(justify right)
+		)
+	)
+	(hierarchical_label "CMP_{r}"
+		(shape input)
+		(at 180.34 60.96 0)
 		(effects
 			(font
@@
 		)
 	)
-	(hierarchical_label "BW"
-		(shape input)
-		(at 29.21 36.83 180)
-		(effects
-			(font
-				(size 1.27 1.27)
-			)
-			(justify right)
-		)
-	)
-	(hierarchical_label "~{14MHz}"
-		(shape input)
-		(at 71.12 34.29 180)
-		(effects
-			(font
-				(size 1.27 1.27)
-			)
-			(justify right)
-		)
-	)
-	(hierarchical_label "CMP_{r}"
-		(shape input)
-		(at 180.34 60.96 0)
-		(effects
-			(font
-				(size 1.27 1.27)
-			)
-			(justify left)
-		)
-	)
 	(hierarchical_label "14MHz"
 		(shape input)
-		(at 71.12 90.17 180)
-		(effects
-			(font
+		(at 46.99 90.17 180)
+		(effects
+			(font

Commit message: A little work on composite output and GPIB
Parts:
- added C108: C_Polarized, symbol Device:C_Polarized
- added R54, R55, R56, R57, R62, R63, R64, R75, R76: ??Ω, seequa_footprints:R_Seequa_Resistor, symbol Device:R_Small
Connections:
- net COMPOSITE_OUT: now also C108.1, R64.1
- net GND: now also R62.2, R64.2
- net at U131.16 (O1a): now also R56.1
- net at U131.18 (O0a): now also R55.1
- net at U131.3 (O3b): now also R54.1
- net at U131.5 (O2b): now also R57.1
- new net: C108.2, R63.1
- new net VIDEO_OUT: R62.1, R63.2
