File: kicad/dma.kicad_sch (KiCad schematic)
At the start: 8 parts, among them U103 74LS245, U104 74LS373, U61 8237, U89 74LS04, U99 PAL16R4

Commit message: Fixes to clocks,  keyboard controller stuff.
Connections:
- net RESET renamed RESET_{BRD}
- net ~{RESET} renamed ~{RESET_{BRD}}
Changed lines of the file:
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@@
 		)
 	)
-	(global_label "~{RESET}"
+	(global_label "~{RESET_{BRD}}"
 		(shape input)
 		(at 30.48 101.6 180)
@@
 		)
 	)
-	(global_label "RESET"
+	(global_label "RESET_{BRD}"
 		(shape input)
 		(at 54.61 101.6 0)

Commit message: update kicad project
Parts:
- removed unit 5 of U89
- removed unit 1 of U89
- removed unit 6 of U89
- added R74B1: R_Small, seequa_footprints:R_Seequa_Resistor, symbol Device:R_Small
- added U102: 74LS74, Package_DIP:DIP-14_W7.62mm, symbol 74xx:74LS74
- added U108: 74LS393, Package_DIP:DIP-14_W7.62mm, symbol 74xx:74LS393
- added U127: 74LS125, Package_DIP:DIP-14_W7.62mm, symbol 74xx:74LS125
- added U128: 74LS175, Package_DIP:DIP-16_W7.62mm, symbol 74xx:74LS175
- R12: seq_coord (none) -> L11; seq_silkscreen (none) -> RN12
- R73, R74: seq_coord (none) -> K9
- U103: seq_coord (none) -> L6
- U104: seq_coord (none) -> L7
- U61: seq_coord (none) -> K10; seq_silkscreen (none) -> 8237
- U89: seq_coord (none) -> L11; seq_silkscreen (none) -> LS04
- U99: symbol Logic_Programmable:PAL16R8 -> seequa:PAL16R4; seq_coord (none) -> M3
Connections:
- net +5V: now also U102.10 (~{S}), U102.12 (D), U128.1 (~{Mr}), U128.16 (VCC)
- net DACK_{0}: now also U102.13 (~{R})
- net DCLK: now also U108.1 (CP), U128.9 (Cp)
- net DMA_AD2: now also R74B1.2; no longer U103.13 (B5)
- net DMA_{READY}: now also U128.7 (Q1)
- net DRQ_{0}: now also U102.9 (Q)
- net GND: now also U127.12, U127.4, U128.8 (GND)
- net DCON_S renamed ~{88_PRIMARY}
- net DMA_AD0_{t} renamed DMA_AD0'
- net DMA_AD1_{t} renamed DMA_AD1'
- net ~{PBUS_{AEN}} renamed PBUS_{DIR}
- net ~{U127D_{EN}} renamed ~{BUS_WAIT}
- net ~{BUS_WAIT}: now also U127.13
- net ~{VRAM_{DECODE_Q}} renamed VRAM_{DECODE_Q}
- new net: U102.11 (C), U108.10 (Q1)
- new net: U128.13 (D3), U128.2 (Q0)
- new net: U127.6, U128.5 (D1)
- new net: U108.12 (MR), U108.2 (MR)
- new net: U108.13 (CP), U108.6 (Q3)
- new net DMA_AD2': R74B1.1, U103.13 (B5)
- new net IO_CH_READY: U127.11, U127.5
- new net KBD_{CLK}: U128.4 (D0)
- new net ~{KBD_SHIFT_{CLK}}: U128.14 (~{Q3})
- no-connect marks 1 -> 15
Other:
- moved on the sheet: R73, R74, U89G, U99

Commit message: More updates
Connections:
- net VRAM_{DECODE_Q} renamed VMEM_{DECODE_Q}
Changed lines of the file:
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@@
 		)
 	)
-	(text_box "This creates a clock divisor of /4."
+	(text_box "This 4-bit counter divides DCLK by 4 to produce DRAM refresh timings."
 		(exclude_from_sim no)
-		(at 194.31 208.28 0)
-		(size 38.1 5.08)
+		(at 191.77 208.28 0)
+		(size 38.1 15.24)
 		(margins 0.9525 0.9525 0.9525 0.9525)
 		(stroke
@@
 		)
 	)
-	(text_box "Bodge wiring.\n\nSeequa added two bodge wires between the termination resistors on DMA_AD0 & DMA_AD1 and ran them over to the video unit, cutting the original XA0 and XA1 traces.\nThese net ties are used to create a new bus representing these bodge wires."
+	(text_box "Bodge wiring.\n\nSeequa added two bodge wires between the termination resistors on DMA_AD0 & DMA_AD1 and ran them over to the video unit, cutting the original XA0 and XA1 traces.\nI hsve called these new adress lines \"XAT\" or XA-terminated; additionally I have added a termination resistor for AD2 as well."
 		(exclude_from_sim no)
 		(at 321.31 77.47 0)
@@
 	(wire
 		(pts
-			(xy 279.4 91.44) (xy 292.1 91.44)
+			(xy 279.4 91.44) (xy 293.37 91.44)
 		)
 		(stroke
@@
 	(wire
 		(pts
-			(xy 279.4 93.98) (xy 292.1 93.98)
+			(xy 279.4 93.98) (xy 293.37 93.98)
 		)
 		(stroke
@@
 	(global_label "PBUS_{DIR}"
 		(shape output)
-		(at 292.1 91.44 0)
+		(at 293.37 91.44 0)
 		(fields_autoplaced yes)
 		(effects
@@
 		)
 		(property "Intersheetrefs" "${INTERSHEET_REFS}"
-			(at 302.26 91.44 0)
+			(at 303.53 91.44 0)
 			(effects
 				(font
@@
 		)
 	)
-	(global_label "VRAM_{DECODE_Q}"
+	(global_label "VMEM_{DECODE_Q}"
 		(shape input)
 		(at 240.03 88.9 180)
@@
 	(global_label "~{PBUS_{OE}}"
 		(shape output)
-		(at 292.1 93.98 0)
+		(at 293.37 93.98 0)
 		(fields_autoplaced yes)
 		(effects
@@
 		)
 		(property "Intersheetrefs" "${INTERSHEET_REFS}"
-			(at 302.26 93.98 0)
+			(at 303.53 93.98 0)
 			(effects
 				(font
@@
 			)
 		)
+		(property "seq_port" ""
+			(at 137.16 97.79 0)
+			(effects
+				(font
+					(size 1.27 1.27)
+				)
+				(hide yes)
+			)
+		)
 		(pin "4"
 		)
@@
 			)
 		)
+		(property "seq_port" ""
+			(at 31.75 264.16 0)
+			(effects
+				(font
+					(size 1.27 1.27)
+				)
+				(hide yes)
+			)
+		)
 		(pin "4"
 		)
@@
 			(at 137.16 133.35 0)
 			(effects
+				(font
+					(size 1.27 1.27)
+				)
+				(hide yes)
+			)
+		)
+		(property "seq_port" ""
+			(at 137.16 133.35 0)
+			(effects

Commit message: Add parallel port, game port
Connections:
- net ~{8259_{CS}} renamed ~{8237_{CS}}
Changed lines of the file:
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@@
 		)
 	)
-	(label "~{8259_{CS}}"
+	(label "~{8237_{CS}}"
 		(at 72.39 74.93 0)
 		(effects
