File: kicad/fdc.kicad_sch (KiCad schematic)
At the start: 8 parts, among them J1 Conn_02x17_Odd_Even, U144 DM74LS07N, U156 74LS240, U157 74LS240, U159 74LS393, U160 74LS123, U84 UPD765AC

Commit message: update kicad project
Parts:
- added U165: PAL16L8, Package_DIP:DIP-20_W7.62mm, symbol Logic_Programmable:PAL16L8
- added U171: 74LS221, Package_DIP:DIP-16_W7.62mm, symbol 74xx:74LS221
- added U172: LF351N, Package_DIP:DIP-8_W7.62mm, symbol Amplifier_Operational:LF351N
- added U173: 74LS107, Package_DIP:DIP-14_W7.62mm, symbol 74xx:74LS107
- added U174: 74LS14, Package_DIP:DIP-14_W7.62mm, symbol 74xx:74LS14
- J1: seq_coord (none) -> D34; seq_silkscreen (none) -> J1
- OSC1: seq_coord (none) -> C31
- U144: seq_coord (none) -> E33
- U156: seq_coord (none) -> D33; seq_silkscreen (none) -> LS240
- U157: seq_coord (none) -> E33; seq_silkscreen (none) -> LS240
- U159: seq_coord (none) -> C32; seq_silkscreen (none) -> LS393
- U160: seq_coord (none) -> C29; seq_silkscreen (none) -> LS123
- U84: seq_coord (none) -> D31
Connections:
- net GND: now also OSC1.7 (GND), U144.7 (GND), U156.1 (OEa), U159.2 (MR), U159.7 (GND), U160.9 (A), U165.10 (GND), U171.1 (~{A}), U171.8 (GND), U173.7 (GND), U174.7 (GND)
- net +5V: now reaches OSC1.14 (Vcc)
- net +5V: now also U144.14 (VCC), U156.20 (VCC), U157.20 (VCC), U159.14 (VCC), U160.11 (Clr), U160.16 (VCC), U160.3 (Clr), U84.40 (Vcc), U165.20 (V_{CC}), U171.16 (VCC), U172.7 (V+), U173.14 (VCC), U173.8 (J), U174.14 (VCC)
- net DCLK: now reaches U159.4 (Q1)
- net T/C: now reaches U84.16 (TC)
- net FDC_{VCO}: now reaches U84.24 (VCO)
- net FDC_{VCO}: now also U171.3 (~{CLR})
- net ~{XIOW}: now reaches U84.3 (~{WR})
- net ~{XIOW}: now also U165.9 (I_{8})
- net XAT0: now reaches U84.5 (A0)
- net XD0 renamed PD0
- net PD0: now also U165.2 (I_{1})
- net XD1 renamed PD1
- net XD2 renamed PD2
- net PD2: now also U165.7 (I_{6})
- net XD3 renamed PD3
- net XD4 renamed PD4
- net PD4: now also U165.6 (I_{5})
- net XD5 renamed PD5
- net PD5: now also U165.3 (I_{2})
- net XD6 renamed PD6
- net XD7 renamed PD7
- net ~{IOR} renamed ~{XIOR}
- new net: U174.11, U174.8
- new net: U173.10 (~{R}), U173.12 (C), U174.12
- new net: U173.5 (Q), U174.1
- new net: U173.13 (~{R}), U173.9 (C)
- new net: U173.2 (~{Q}), U174.3
- new net ~{FDC_{CS}}: U165.11 (I_{9})
Other:
- title: (none) -> Floppy Disk Controller
- moved on the sheet: OSC1, U144A, U144B, U144C, U144D, U144E, U144G, U159A, U159B, U159C, U160C, U84

Commit message: Add parallel port, game port
Parts:
- added C85: C_Bypass_5mm, seequa_footprints:C_Seequa_Bypass_Film_5mm, symbol seequa:C_Bypass_Film_2.54mm
Changed lines of the file:
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@@
+	)
+	(symbol
+		(lib_id "seequa:C_Bypass_Film_2.54mm")
+		(at 207.01 354.33 0)
+		(unit 1)
+		(exclude_from_sim no)
+		(in_bom yes)
+		(on_board yes)
+		(dnp no)
+		(property "Reference" "C85"
+			(at 208.9864 353.2549 90)
+			(effects
+				(font
+					(size 1.27 1.27)
+				)
+				(justify left)
+			)
+		)
+		(property "Value" "C_Bypass_5mm"
+			(at 207.264 356.362 0)
+			(effects
+				(font
+					(size 1.27 1.27)
+				)
+				(justify left)
+				(hide yes)
+			)
+		)
+		(property "Footprint" "seequa_footprints:C_Seequa_Bypass_Film_5mm"
+			(at 207.518 364.998 0)
+			(effects
+				(font
+					(size 1.27 1.27)
+				)
+				(hide yes)
+			)
+		)
+		(property "Datasheet" "~"
+			(at 207.01 354.33 0)
+			(effects
+				(font
+					(size 1.27 1.27)
+				)
+				(hide yes)
+			)
+		)
+		(property "Description" "0.1uF Dipped Film, ±10%"
+			(at 219.964 358.394 0)
+			(effects
+				(font
+					(size 1.27 1.27)
+				)
+				(hide yes)
+			)
+		)
+		(property "seq_partno" ""
+			(at 207.01 354.33 0)
+			(effects
+				(font
+					(size 1.27 1.27)
+				)
+				(hide yes)
+			)
+		)
+		(property "seq_coord" ""
+			(at 207.01 354.33 0)
+			(effects
+				(font
+					(size 1.27 1.27)
+				)
+				(hide yes)
+			)
+		)
+		(property "seq_silkscreen" ""
+			(at 207.01 354.33 0)
+			(effects
+				(font
+					(size 1.27 1.27)
+				)
+				(hide yes)
+			)
+		)
+		(property "seq_sharpie" ""
+			(at 207.01 354.33 0)
+			(effects
+				(font
+					(size 1.27 1.27)
+				)
+				(hide yes)
+			)
+		)
+		(property "seq_notes" ""
+			(at 207.01 354.33 0)
+			(effects
+				(font
+					(size 1.27 1.27)
+				)
+				(hide yes)
+			)
+		)
+		(property "seq_port" ""
+			(at 207.01 354.33 0)
+			(effects
+				(font
+					(size 1.27 1.27)
+				)
+				(hide yes)
+			)
+		)
+		(pin "2"
+		)
+		(pin "1"
+		)
+		(instances
+			(project "seequa_chameleon"
+				(path "/ae890d4c-6a02-4621-80ce-7ef4317218ea/458f4203-88af-4514-ba76-e86555deb564"
+					(reference "C85")
+					(unit 1)
+				)
+			)
+		)
 	)
 	(symbol

Commit message: Updates, chameleon logo
Connections:
- net +5V: now also C85.1
- net GND: now also C85.2
Changed lines of the file:
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@@
 		(title "Floppy Disk Controller")
 	)
+	(text_box "Omitted from motherboard, so value is unknown."
+		(exclude_from_sim no)
+		(at 212.09 355.6 0)
+		(size 16.51 10.16)
+		(margins 0.9525 0.9525 0.9525 0.9525)
+		(stroke
+			(width 0)
+			(type solid)
+		)
+		(fill
+			(type color)
+			(color 255 229 191 1)
+		)
+		(effects
+			(font
+				(face "Arial")
+				(size 1.27 1.27)
+			)
+			(justify left top)
+		)
+	)
 	(junction
 		(at 220.98 153.67)
@@
 	(junction
 		(at 238.76 153.67)
+		(diameter 0)
+		(color 0 0 0 0)
+	)
+	(junction
+		(at 171.45 339.09)
 		(diameter 0)
 		(color 0 0 0 0)
@@
 	(wire
 		(pts
+			(xy 207.01 356.87) (xy 207.01 369.57)
+		)
+		(stroke
+			(width 0)
+			(type default)
+		)
+	)
+	(wire
+		(pts
 			(xy 161.29 74.93) (xy 161.29 77.47)
 		)
@@
 	(wire
 		(pts
+			(xy 207.01 351.79) (xy 207.01 339.09)
+		)
+		(stroke
+			(width 0)
+			(type default)
+		)
+	)
+	(wire
+		(pts
 			(xy 250.19 118.11) (xy 228.6 118.11)
 		)
@@
 	(wire
 		(pts
+			(xy 207.01 339.09) (xy 171.45 339.09)
+		)
+		(stroke
+			(width 0)
+			(type default)
+		)
+	)
+	(wire
+		(pts
 			(xy 212.09 227.33) (xy 226.06 227.33)
 		)
@@
 		)
 		(stroke
+			(width 0)
+			(type default)
+		)
+	)
+	(wire
+		(pts
+			(xy 207.01 369.57) (xy 171.45 369.57)
+		)
+		(stroke
