File: kicad/io_decode.kicad_sch (KiCad schematic)
At the start: 2 parts, among them U101 PAL20L10, U118 74LS138

Commit message: update kicad project
Parts:
- U101: seq_coord (none) -> M6
- U118: seq_coord (none) -> M25
Connections:
- net ~{FDC_{CS}}: now reaches U101.15 (I/~{O_{2}})
- no-connect marks 1 -> 2

Commit message: Updates, chameleon logo
Connections:
- net ~{VIDEO_DECODER_{CS}} renamed ~{VIDEO_DECODER_{EN}}
Changed lines of the file:
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@@
 		)
 	)
-	(label "~{VIDEO_DECODER_{CS}}"
+	(label "~{VIDEO_DECODER_{EN}}"
 		(at 140.97 95.25 180)
 		(effects
