File: kicad/p_bus.kicad_sch (KiCad schematic)
At the start: 1 part, among them U66 74LS245

Commit message: update kicad project
Parts:
- U66: seq_coord (none) -> H17; seq_silkscreen (none) -> LS245
Connections:
- net ~{PBUS_{AEN}} renamed PBUS_{DIR}
