File: kicad/parallel.kicad_sch (KiCad schematic)
At the start: 14 parts, among them J8 LPT_IDC, U152 74LS155, U153 74LS367, U166 74LS05, U167 74LS174, U168 74LS240

Commit message: update kicad project
Parts:
- added U143: 74LS244, Package_DIP:DIP-20_W7.62mm, symbol 74xx:74LS244
- added unit 7 of U166
- added unit 5 of U166
- added unit 4 of U166
- added unit 1 of U166
- added unit 2 of U166
- added unit 6 of U166
- added U169: 74LS374, Package_DIP:DIP-20_W7.62mm, symbol 74xx:74LS374
- added U175: 74LS04, Package_DIP:DIP-14_W7.62mm, symbol 74xx:74LS04
- C73, C74, C75, C76, C77, C78: seq_coord (none) -> H25
- C79, C80: seq_coord (none) -> G25
- J8: seq_coord (none) -> H26
- U152: seq_coord (none) -> I23
- U153: seq_coord (none) -> I24
- U166: seq_coord (none) -> J26; seq_silkscreen (none) -> LS05
- U167: seq_coord (none) -> I26; seq_notes (none) -> LPT Control Register; seq_silkscreen (none) -> LS174
- U168: seq_coord (none) -> I28; seq_silkscreen (none) -> LS240
Connections:
- net NMI_P2 is gone; now on net LPT_SELECT_IN: U153.10 (I4)
- net +5V: now also U167.16 (VCC), U168.20 (VCC), U143.20 (VCC), U169.20 (VCC)
- net GND: now also U143.10 (GND), U169.10 (GND)
- net PD3: now also U168.9 (O0b)
- net PD4: now also U167.14 (D5), U168.18 (O0a)
- net PD5: now also U168.7 (O1b)
- net PD6: now also U168.14 (O2a)
- net PD7: now also U168.12 (O3a)
- net ~{LPT_CONTROL_{CS}}: now also U167.9 (Cp)
- net ~{LPT_DATA_{CS}}: now also U143.19 (OEb)
- net S_ERROR: now reaches U153.12 (I5)
- net PD2: now reaches U153.13 (O6b)
- net PD2: now also U167.13 (D4), U168.16 (O1a), U168.5 (O2b)
- net S_IRQ: now reaches U153.14 (I6)
- net S_PAPER_OUT: now reaches U153.6 (I3)
- net XAT0: now reaches U152.13 (A0)
- net XAT1: now reaches U152.3 (A1)
- net LPT_SELECT_IN: now reaches U168.3 (O3b)
- net LPT_SELECT_IN: now also U169.8 (D3)
- net BUSY: now reaches U168.8 (I3a)
- net BUSY: now also J8.21 (BUSY)
- net ~{STB}: now reaches J8.1 (~{STB})
- net ~{STB}: now also U166.6
- net ~{ACK}: now reaches J8.19 (~{ACK})
- net ~{ACK}: now also U175.1
- net ~{AFD}: now reaches J8.2 (~{AFD})
- net ~{AFD}: now also U166.4
- net PE: now reaches J8.23 (PE)
- net SELECT: now reaches J8.25 (SLCT)
- net ~{ERR}: now reaches J8.4 (~{ERR})
- net ~{INIT}: now reaches J8.6 (~{INIT})
- net ~{INIT}: now also U166.2
- net ~{SELECT_IN}: now reaches J8.8 (~{SLIN})
- net ~{SELECT_IN}: now also U166.10
- net ~{RESET_{BRD}}: now reaches U167.1 (~{Mr})
- net C_SELECT: now reaches U167.10 (Q3)
- net C_SELECT: now also U166.11
- net ~{C_INIT}: now reaches U167.12 (Q4)
- net ~{C_INIT}: now also U166.9
- net C_IRQ_{EN}: now reaches U167.15 (Q5)
- net C_STB: now reaches U166.5, U167.2 (Q0)
- net BIDI: now reaches U167.5 (Q1)
- net C_AFD: now reaches U167.7 (Q2)
- net C_AFD: now also U166.3
- net NMI_P16 renamed ~{LPT_S_ACK}
- new net: U166.1, U166.8
- new net: U143.18 (O0a), U169.3 (D0)
- new net: U143.15 (I2b), U169.5 (O1)
- new net: U143.14 (O2a), U169.7 (D2)
- new net LPT_IRQACK: U175.2
Other:
- moved on the sheet: U168

Commit message: More updates
Parts:
- U175: seq_silkscreen (none) -> LS04
Connections:
- net LPT_SELECT_IN: no longer U153.10 (I4)
- net S_PAPER_OUT: no longer U153.6 (I3)
Changed lines of the file:
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@@
 		)
 	)
-	(label "S_BUSY"
-		(at 181.61 36.83 0)
-		(effects
-			(font
-				(size 1.27 1.27)
-			)
-			(justify left bottom)
-		)
-	)
 	(label "~{C_INIT}"
 		(at 27.94 161.29 0)
@@
 		)
 	)
+	(label "S_BUSY"
+		(at 172.72 21.59 0)
+		(effects
+			(font
+				(size 1.27 1.27)
+			)
+			(justify left bottom)
+		)
+	)
 	(label "PD5"
 		(at 111.76 93.98 0)
@@
 	)
 	(label "S_SELECT_IN"
-		(at 181.61 44.45 0)
-		(effects
-			(font
-				(size 1.27 1.27)
-			)
-			(justify left bottom)
-		)
-	)
-	(label "S_SELECT_IN"
 		(at 234.95 107.95 180)
 		(effects
@@
 		)
 	)
+	(label "S_PAPER_OUT"
+		(at 172.72 26.67 0)
+		(effects
+			(font
+				(size 1.27 1.27)
+			)
+			(justify left bottom)
+		)
+	)
 	(label "XAT0"
 		(at 52.07 62.23 0)
@@
 	)
 	(label "S_ACK"
-		(at 181.61 39.37 0)
+		(at 172.72 24.13 0)
 		(effects
 			(font
@@
 		)
 	)
-	(label "S_PAPER_OUT"
-		(at 181.61 41.91 0)
-		(effects
-			(font
-				(size 1.27 1.27)
-			)
-			(justify left bottom)
-		)
-	)
 	(label "S_ERROR"
 		(at 181.61 46.99 0)
@@
 		)
 	)
+	(label "S_SELECT_IN"
+		(at 172.72 29.21 0)
+		(effects
+			(font
+				(size 1.27 1.27)
+			)
+			(justify left bottom)
+		)
+	)
 	(global_label "~{LPT_S_ACK}"
 		(shape input)
@@
 			)
 		)
-		(property "seq_silkscreen" ""
+		(property "seq_silkscreen" "LS04"
 			(at 58.42 251.46 0)
 			(effects
@@
 			)
 		)
-		(property "seq_silkscreen" ""
+		(property "seq_silkscreen" "LS04"
 			(at 280.67 218.44 0)
 			(effects
@@
 			)
 		)
-		(property "seq_silkscreen" ""
+		(property "seq_silkscreen" "LS04"
 			(at 287.02 177.8 0)
 			(effects
@@
 			)
 		)
-		(property "seq_silkscreen" ""
+		(property "seq_silkscreen" "LS04"
 			(at 285.75 198.12 0)
 			(effects
@@
 			)
 		)
-		(property "seq_silkscreen" ""
+		(property "seq_silkscreen" "LS04"
 			(at 276.86 251.46 0)
 			(effects
@@
 			)
 		)
-		(property "seq_silkscreen" ""
+		(property "seq_silkscreen" "LS04"
 			(at 281.94 236.22 0)
 			(effects
@@
 			)
 		)
-		(property "seq_silkscreen" ""
+		(property "seq_silkscreen" "LS04"
 			(at 195.58 160.02 0)
 			(effects

Commit message: Add parallel port, game port
Parts:
- removed unit 4 of U175
- removed unit 5 of U175
- added C81: C_Small, seequa_footprints:C_Seequa_Bypass_6.5mm, symbol Device:C_Small
- added RN13: R_Network05_Split, Resistor_THT:R_Array_SIP6, symbol Device:R_Network05_Split
- U153: seq_notes LPT Status Register -> LPT Read Register 0
- U167: seq_notes LPT Control Register -> LPT Control Write Register
- U168: seq_notes (none) -> LPT Read Register 1
Connections:
- net C_IRQ_{EN} is gone; now on net LPT_IRQ_EN: U167.15 (Q5)
- net S_ERROR is gone; now on net ~{ERR}: U153.12 (I5)
- net ~{LPT_DATA_{CS}} is gone; now on net ~{LPT_DATA_{RD}}: U143.19 (OEb), U152.7 (Q0a)
- net ~{LPT_STATUS_{CS2}} is gone; now on net ~{LPT_CONTROL_{RD}}: U152.5 (Q2a), U153.1 (OEa)
- net +5V: now also U166.14 (VCC), U175.14 (VCC), RN13.1 (R1), RN13.1 (R1), RN13.1 (R1), RN13.1 (R1), RN13.1 (R1)
- net BUSY: no longer U168.8 (I3a)
- net GND: now also U166.7 (GND), U169.1 (OE), U175.7 (GND), C81.2
- net LPT_SELECT_IN: no longer U168.3 (O3b), U169.8 (D3)
- net PD0: now also U143.9 (O0b), U168.3 (O3b), U169.8 (D3)
- net PD1: now also U143.3 (O3b), U169.18 (D7)
- net PD2: now also U143.14 (O2a), U169.7 (D2); no longer U168.16 (O1a)
- net PD3: now also U143.16 (O1a), U169.17 (D6)
- net PD4: now also U143.5 (O2b), U169.4 (D1)
- net PD5: now also U143.7 (O1b), U168.16 (O1a), U169.14 (D5)
- net PD6: now also U143.18 (O0a), U169.3 (D0)
- net PD7: now also U143.12 (O3a), U169.13 (D4)
- net PE: now also U175.3
- net SELECT: now also U175.5
- net ~{AFD}: now also U168.13 (I1b), RN13.4 (R3.2)
- net ~{INIT}: now also U166.13, RN13.2 (R1.2)
- net ~{SELECT_IN}: now also U168.11 (I0b)
- net ~{STB}: now also U168.17 (I3b), C81.1, RN13.5 (R4.2)
- net LD3: now reaches C76.1, J8.9 (PD3)
- net LD3: now also U143.4 (I1a), U169.16 (O6)
- net LD1: now reaches C74.1, J8.5 (PD1)
- net LD1: now also U143.17 (I3b), U169.19 (O7)
- net LD2: now reaches C75.1, J8.7 (PD2)
- net LD2: now also U143.6 (I2a), U169.6 (O2)
- net LPT_IRQ_EN: now reaches U153.10 (I4)
- net INT: now reaches U153.6 (I3)
- net S_PE: now reaches U175.4
- net S_PE: now also U168.4 (I1a)
- net S_SELECT: now reaches U175.6
- net S_SELECT: now also U168.2 (I0a)
- net ~{LPT_DATA_{WR}}: now reaches U152.9 (Q0b)
- net ~{LPT_DATA_{WR}}: now also U169.11 (Cp)
- net INIT': now reaches U166.1, U166.8
- net INIT': now also RN13.6 (R5.2)
- net LD7: now reaches C80.2, J8.17 (PD7)
- net LD7: now also U143.8 (I3a), U169.12 (O4)
- net LD5: now reaches U169.15 (O5)
- net LD5: now also C78.1, J8.13 (PD5), U143.13 (I1b)
- net LD6: now reaches U169.2 (O0)
- net LD6: now also C79.1, J8.15 (PD6), U143.2 (I0a)
- net LD4: now reaches U143.15 (I2b), U169.5 (O1)
- net LD4: now also C77.1, J8.11 (PD4)
- net LD0: now reaches U169.9 (O3)
- net LD0: now also C73.1, J8.3 (PD0), U143.11 (I0b)
- net INIT: now reaches U168.15 (I2b)
- net INIT: now also U166.12, RN13.3 (R2.2)
- net ~{LPT_CONTROL_{RD}}: now reaches U168.19 (OEb)
- net ~{S_ACK}: now reaches U168.6 (I2a)
- net ~{LPT_DATA_{RD}}: now reaches U143.1 (OEa)
- net C_SELECT renamed C_SELECT_IN
- net LPT_IRQACK renamed LPT_ACK
- net ~{LPT_CONTROL_{CS}} renamed ~{LPT_CONTROL_{WR}}
- net ~{LPT_S_ACK} renamed ~{IO_NMI}
- new net ~{S_BUSY}: U168.8 (I3a)
- no-connect marks 0 -> 2
Other:
- note added: "LPT Control Register - 37Eh"
- note added: "LPT Status Register - 37Dh"
- note added: "To NMI control PAL (page 2)"
- note added: "To Parallel Port"
- note added: "To U168 Control Readback Register"
- title: (none) -> Parallel Port
- moved on the sheet: C73, C74, C75, C76, C77, C78, C79, C80, J8, U143, U166A, U166B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

Commit message: Updates, chameleon logo
Connections:
- net INT renamed INT_{87}
Changed lines of the file:
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@@
 		)
 	)
-	(global_label "INT"
+	(global_label "INT_{87}"
 		(shape input)
 		(at 170.18 41.91 180)
