File: kicad/parts.kicad_sch (KiCad schematic)
At the start: 11 parts, among them J14 Power Connector, U102 74LS74, U108 74LS393, U141 74LS74, U62 74LS08, U82 74LS00

Commit message: update kicad project
Parts:
- removed unit 2 of U102
- removed unit 2 of U108
- removed unit 1 of U108
- added R10: ??Ω, seequa_footprints:R_Seequa_Resistor, symbol Device:R_Small
- C100, C119: seq_coord (none) -> L4
- C120: seq_coord (none) -> C31
- C93: seq_coord (none) -> H20
- C94: seq_coord (none) -> J15
- J14: seq_coord (none) -> M32; seq_silkscreen (none) -> J14
- U102: seq_coord (none) -> L5; seq_silkscreen (none) -> LS74
- U108: seq_coord (none) -> D16; seq_silkscreen (none) -> LS393
- U141: seq_coord (none) -> I15; seq_silkscreen (none) -> LS74
- U62: seq_coord (none) -> B10; seq_silkscreen (none) -> LS08
- U82: seq_coord (none) -> D20; seq_silkscreen (none) -> LS00
Other:
- moved on the sheet: C100, C119, C120, C93, C94, J14, U102A, U102C, U108C, U62B, U82E
