File: kicad/pit.kicad_sch (KiCad schematic)
At the start: 1 part, among them U59 8253

Commit message: update kicad project
Parts:
- U59: seq_coord (none) -> H13; seq_silkscreen (none) -> 8253
Connections:
- net +5V: now also U59.11 (G0), U59.14 (G1)
- net ~{IOR} renamed ~{XIOR}
- net ~{IOW} renamed ~{XIOW}

Commit message: Add parallel port, game port
Connections:
- net XA0 renamed XAT0
- net XA1 renamed XAT1
Changed lines of the file:
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@@
-	)
-	(bus_entry
-		(at 86.36 102.87)
-		(size 2.54 2.54)
-		(stroke
-			(width 0)
-			(type default)
-		)
 	)
 	(bus_entry
@@
 	)
 	(bus_entry
+		(at 119.38 102.87)
+		(size 2.54 2.54)
+		(stroke
+			(width 0)
+			(type default)
+		)
+	)
+	(bus_entry
 		(at 121.92 74.93)
 		(size 2.54 2.54)
@@
 	(bus_entry
 		(at 119.38 97.79)
-		(size 2.54 2.54)
-		(stroke
-			(width 0)
-			(type default)
-		)
-	)
-	(bus_entry
-		(at 86.36 105.41)
 		(size 2.54 2.54)
 		(stroke
@@
 		)
 	)
+	(bus_entry
+		(at 119.38 105.41)
+		(size 2.54 2.54)
+		(stroke
+			(width 0)
+			(type default)
+		)
+	)
 	(wire
 		(pts
@@
 		)
 		(stroke
-			(width 1)
+			(width 0.75)
 			(type default)
 			(color 194 194 0 1)
@@
 		)
 		(stroke
-			(width 1)
+			(width 0.75)
 			(type default)
 			(color 0 194 194 1)
@@
 		)
 		(stroke
-			(width 1)
+			(width 0.75)
 			(type default)
 			(color 0 194 194 1)
@@
 		)
 		(stroke
-			(width 1)
+			(width 0.75)
 			(type default)
 			(color 0 194 194 1)
@@
 	(wire
 		(pts
-			(xy 88.9 105.41) (xy 137.16 105.41)
+			(xy 121.92 107.95) (xy 137.16 107.95)
 		)
 		(stroke
@@
 	(bus
 		(pts
-			(xy 86.36 102.87) (xy 86.36 105.41)
-		)
-		(stroke
-			(width 1)
-			(type default)
-		)
-	)
-	(bus
-		(pts
 			(xy 119.38 97.79) (xy 119.38 100.33)
 		)
 		(stroke
-			(width 1)
+			(width 0.75)
 			(type default)
 			(color 0 0 194 1)
@@
 		)
 		(stroke
-			(width 1)
+			(width 0.75)
 			(type default)
 			(color 0 194 194 1)
@@
 		)
 		(stroke
-			(width 1)
+			(width 0.75)
 			(type default)
 			(color 132 0 132 1)
@@
 		)
 		(stroke
-			(width 1)
-			(type default)
-			(color 0 194 194 1)
-		)
-	)
-	(bus
-		(pts
-			(xy 85.09 102.87) (xy 86.36 102.87)
-		)
-		(stroke
-			(width 1)
-			(type default)
+			(width 0.75)
+			(type default)
+			(color 0 194 194 1)
 		)
 	)
@@
 		)
 		(stroke
-			(width 1)
+			(width 0.75)
 			(type default)
 			(color 0 194 194 1)
@@
 		)
 		(stroke
-			(width 1)
+			(width 0.75)
 			(type default)
 			(color 132 0 132 1)
@@
 	(wire
 		(pts
-			(xy 88.9 107.95) (xy 137.16 107.95)
-		)
-		(stroke
-			(width 0)
-			(type default)
-		)
-	)
-	(wire
-		(pts
 			(xy 124.46 80.01) (xy 137.16 80.01)
 		)
@@
 		)
 	)
+	(bus
+		(pts
+			(xy 119.38 100.33) (xy 119.38 102.87)
+		)
+		(stroke
+			(width 0.75)
+			(type default)
+			(color 0 0 194 1)
+		)
+	)
 	(wire
 		(pts
@@
 	(wire
 		(pts
+			(xy 121.92 105.41) (xy 137.16 105.41)
+		)
+		(stroke
+			(width 0)
+			(type default)
+		)
+	)
+	(wire
+		(pts
 			(xy 157.48 107.95) (xy 170.18 107.95)
 		)
@@
 		)
 		(stroke
-			(width 1)
+			(width 0.75)
 			(type default)
 			(color 0 194 194 1)
@@
 		)
 		(stroke
-			(width 1)
+			(width 0.75)
 			(type default)
 			(color 0 194 194 1)
@@
 		)
 		(stroke
-			(width 1)
+			(width 0.75)
 			(type default)
 			(color 0 0 194 1)
@@
 		)
 		(stroke
-			(width 1)
+			(width 0.75)
 			(type default)
 			(color 0 194 194 1)
@@
 	(bus
 		(pts
+			(xy 119.38 102.87) (xy 119.38 105.41)
+		)
+		(stroke
+			(width 0.75)
+			(type default)
+			(color 0 0 194 1)
+		)
+	)
+	(bus
+		(pts
 			(xy 85.09 87.63) (xy 119.38 87.63)
 		)
 		(stroke
-			(width 1)
+			(width 0.75)
 			(type default)
 			(color 0 0 194 1)
@@
 		)
 	)
-	(label "XA1"
-		(at 127 107.95 0)
-		(effects
-			(font
-				(size 1.27 1.27)
-			)
-			(justify left bottom)
-		)
-	)
 	(label "~{XIOR}"
 		(at 127 100.33 0)
@@
 		)
 	)
-	(label "XA0"
-		(at 127 105.41 0)
-		(effects
-			(font
-				(size 1.27 1.27)
-			)
-			(justify left bottom)
-		)
-	)
 	(label "PD4"
 		(at 127 87.63 0)
@@
 		)
 	)
+	(label "XAT1"
+		(at 127 107.95 0)
+		(effects
+			(font
+				(size 1.27 1.27)
+			)
+			(justify left bottom)
+		)
+	)
 	(label "PD7"
 		(at 127 95.25 0)
+		(effects
+			(font
+				(size 1.27 1.27)
+			)
+			(justify left bottom)
+		)
+	)
+	(label "XAT0"
+		(at 127 105.41 0)
 		(effects
 			(font
@@
 		(effects
 			(font
-				(size 1.27 1.27)
-			)
-			(justify right)
-		)
-	)
-	(hierarchical_label "XA[0..19]"
-		(shape input)
-		(at 85.09 102.87 180)
-		(effects
-			(font
