File: kicad/video.kicad_sch (KiCad schematic)
At the start: 43 parts, among them J11 Conn_02x05e, U107 74LS157, U109 74LS166, U111 PAL18L4CNS, U112 74LS393, U113 74LS670, U114 74F374, U115 74LS670, U116 74LS107, U117 74F04, U121 74LS166, U123 74LS166, U126 74LS138, U127 74LS125, U128 74LS175, U129 74LS221, U130 74LS221, U131 74LS240, U132 74LS74, U133 74LS74, U134 74LS74, U135 74F374, U136 74LS04, U137 74S374N, U138 74LS368, U139 74LS86, U140 74LS367, U146 PAL18L4, U147 74LS174, U148 74LS174, U149 74LS175, U151 PAL20L2, U154 74LS161, U155 74LS10, U158 PAL20L10, U161 PAL16R6, U166 74LS05, U58 HD46505SP, U65 74LS245, U67 74LS374, U68 74LS244, U82 74LS00, U98 DMPAL12L6NC

Commit message: update kicad project
Parts:
- removed U113, U115: 74LS670, Package_DIP:DIP-16_W7.62mm, symbol 74xx:74LS670
- removed unit 5 of U117
- removed unit 2 of U127
- removed unit 4 of U127
- removed U128, U149: 74LS175, Package_DIP:DIP-16_W7.62mm, symbol 74xx:74LS175
- removed unit 1 of U136
- removed U140: 74LS367, Package_DIP:DIP-16_W7.62mm, symbol 74xx:74LS367
- removed U147, U148: 74LS174, Package_DIP:DIP-16_W7.62mm, symbol 74xx:74LS174
- removed U166: 74LS05, Package_DIP:DIP-14_W7.62mm, symbol 74xx:74LS05
- removed U65: 74LS245, Package_DIP:DIP-20_W7.62mm, symbol 74xx:74LS245
- removed U67: 74LS374, Package_DIP:DIP-20_W7.62mm, symbol 74xx:74LS374
- removed U68: 74LS244, Package_DIP:DIP-20_W7.62mm, symbol 74xx:74LS244
- removed U82: 74LS00, Package_DIP:DIP-14_W7.62mm, symbol 74xx:74LS00
- added U89: 74LS04, Package_DIP:DIP-14_W7.62mm, symbol 74xx:74LS04
- J11: seq_coord (none) -> K28
- U107: seq_coord (none) -> D16; seq_silkscreen (none) -> LS157
- U109: seq_coord (none) -> E16
- U111: seq_coord (none) -> E20; seq_notes (none) -> Character Color MUX
- U112: seq_coord (none) -> F22; seq_notes (none) -> Blink Clock; seq_silkscreen (none) -> LS393
- U114: seq_coord (none) -> H20; seq_notes (none) -> Color Latch (x2)
- U116: seq_coord (none) -> L20; seq_silkscreen (none) -> LS107
- U117: seq_coord (none) -> L20
- U121: seq_coord (none) -> I20
- U123: seq_coord (none) -> I21
- U126: seq_coord (none) -> J15; seq_notes (none) -> Video IO Sub-decoder; seq_silkscreen (none) -> LS138
- U127: seq_coord (none) -> J16; seq_silkscreen (none) -> LS125
- U129, U130: seq_coord (none) -> K32; seq_silkscreen (none) -> LS221
- U131: seq_coord (none) -> J29; seq_silkscreen (none) -> LS240
- U132: seq_coord (none) -> K24; seq_silkscreen (none) -> LS74
- U133: seq_coord (none) -> K25; seq_silkscreen (none) -> LS74
- U134: seq_coord (none) -> I22
- U135: seq_coord (none) -> L28
- U136: seq_coord (none) -> F23; seq_silkscreen (none) -> LS04
- U137: seq_coord (none) -> L22; seq_silkscreen (none) -> S374N
- U138: seq_coord (none) -> K29; seq_silkscreen (none) -> LS368
- U139: seq_coord (none) -> K30; seq_silkscreen (none) -> LS86
- U146: seq_coord (none) -> L23
- U151: seq_coord (none) -> K26
- U154: seq_coord (none) -> H23; seq_silkscreen (none) -> LS161
- U155: seq_coord (none) -> F22; seq_silkscreen (none) -> LS10
- U158: seq_coord (none) -> L21; seq_notes (none) -> Video Memory Controller
- U161: seq_coord (none) -> J21; seq_notes (none) -> Timing Control
- U58: seq_coord (none) -> L16
- U98: seq_coord (none) -> M2; seq_notes Video Address Decoder -> Video Address Decoder PAL
Connections:
- net BODGE0 is gone; now on net C1_{BODGE_OUT}: U146.3 (I_{2})
- net CC_{PAL} is gone; now on net CURSOR_BLINK: U111.1 (I_{0}), U112.6 (Q3)
- net VMUX_{EN} is gone; now on net ~{VMUX_{CRT}}: U158.5 (I_{4})
- net ~{CGA_AEN} is gone; now on net ~{VM_{WR}}: U98.14 (~{O_{2}})
- net ~{OSC} is gone; now on net ~{14MHz}: U117.8, U132.3 (C), U133.3 (C), U137.11 (Cp)
- net ~{SRAM_WR_TIMING} is gone; now on net ~{SRAM_{WE_STR}}: U136.4
- net ~{SRAM_{MR}} is gone; now on net ~{SRAM_{RD}}: U107.7 (Zb)
- net ~{VM_{RAS}'} is gone; now on net ~{VM_{RAS}}: U137.13 (D4), U158.14 (~{O_{1}})
- net +5V: now also U111.24 (V_{CC}), U134.1 (~{R})
- net AT_D0: no longer U121.10 (E)
- net AT_D1: no longer U123.10 (E)
- net AT_D2: now also U111.14 (I_{11}); no longer U111.8 (I_{7}), U123.14 (H)
- net AT_D3: now also U111.13 (I_{13}); no longer U111.14 (I_{11}), U121.11 (F), U123.11 (F)
- net AT_D4: no longer U121.12 (G)
- net AT_D5: no longer U123.12 (G)
- net AT_D6: no longer U121.14 (H)
- net AT_D7: now also U111.8 (I_{7}); no longer U111.13 (I_{13})
- net BW: now also U139.2, U146.4 (I_{3}), U151.22 (I_{19})
- net CRM_P21: now also U117.4; no longer U117.3, U158.21 (I/~{O_{8}})
- net DEN: now also U89.13
- net DOT_CLK: now also U146.1 (I_{0})
- net GND: now also U112.12 (MR), U112.2 (MR)
- net GRAPHICS: now also U111.22 (I_{17}), U151.2 (I_{1})
- net HIRES_GFX: now also U146.14 (I_{11})
- net MEMW: now also U154.9 (~{PE})
- net ~{BW_GRAPHICS}: now also U146.5 (I_{4})
- net ~{CMX_{O0}_DLY}: now also U146.10 (I_{9})
- net ~{CMX_{O1}_DLY}: now also U146.9 (I_{8})
- net ~{CMX_{O2}_DLY}: now also U146.8 (I_{7})
- net ~{CMX_{O3}_DLY}: now also U146.7 (I_{6})
- net ~{CRM_P21}: now also U117.3, U158.21 (I/~{O_{8}}); no longer U117.4
- net ~{DEN}: now also U89.12
- net ~{U131_QA}: now also U151.6 (I_{5})
- net ~{VM_{CAS_T}}: no longer U158.23 (~{O_{10}})
- net ~{VM_{CAS}}: now also U158.23 (~{O_{10}})
- net ~{VM_{RAS}}: no longer U137.12 (O4)
- net ~{VM_{WR}}: no longer U158.8 (I_{7})
- net at U155.12: now also U111.2 (I_{1})
- net CHG_BLINK: now reaches U155.13
- net CHG_BLINK: now also U112.11 (Q0)
- net at U133.10 (~{S}), U133.4 (~{S}): now also U132.1 (~{R}), U132.4 (~{S}), U133.1 (~{R}), U133.13 (~{R}), U139.3
- net U133_{QA}: now reaches U133.12 (D), U133.5 (Q)
- net U133_{QA}: now also U151.9 (I_{8})
- net ~{14MHz}: now reaches U114.11 (Cp)
- net ~{14MHz}: now also U135.11 (Cp)
- net at U135.13 (D4): no longer U146.1 (I_{0})
- net C1_{BODGE_IN}: now reaches U135.14 (D5)
- net C1_{BODGE_OUT}: now reaches U135.15 (O5)
- net CO_{BODGE_OUT}: now reaches U135.16 (O6)
- net CO_{BODGE_OUT}: now also U146.6 (I_{5})
- net C0_{BODGE_IN}: now reaches U135.17 (D6)
- net C0_{BODGE_IN}: now also U151.1 (I_{0})
- net DEN_{L}: now reaches U135.18 (D7)
- net DEN_{L}: now also U132.9 (Q)
- net DEN_{BODGE}: now reaches U135.19 (O7)
- net DEN_{BODGE}: now also U146.13 (I_{13})
- net ~{CRK_P14'}: now reaches U161.14 (~{O_{3}})
- net ~{CRK_P16'}: now reaches U161.16 (~{O_{5}})
- net ~{CRK_P16'}: now also U137.8 (D3), U158.9 (I_{8})
- net ~{HCLK'}: now reaches U161.17 (~{O_{6}})
- net ~{HCLK'}: now also U137.7 (D2), U158.8 (I_{7})
- net ~{CRK_P18'}: now reaches U137.4 (D1), U158.7 (I_{6}), U161.18 (~{O_{7}})
- net ~{HCLK}: now reaches U158.11 (I_{10}), U161.8 (I_{7})
- net ~{HCLK}: now also U132.2 (D), U137.6 (O2)
- net ~{SRAM_{WE_STR}}: now reaches U107.14 (I0d)
- net ~{CRK_P16}: now reaches U137.9 (O3), U158.10 (I_{9})
- net CURSOR_BLINK: now reaches U112.13 (CP)
- net BG_{B}: now reaches U146.15 (I_{14})
- net BG_{G}: now reaches U146.16 (I_{15})
- net BG_{R}: now reaches U146.21 (I_{16})
- net BG_{I}: now reaches U146.22 (I_{17})
- net VRAM_{EN}: now reaches U151.5 (I_{4})
- net CRM_P20 renamed ~{VM_{RDGATE}}
- net CRM_P22 renamed ~{CRK_P18}
- net CRM_{VA5} renamed CRM_{A12}
- net CURSOR_OUT renamed CURSOR_{L}
- net FG_I renamed FG_{I}
- net MA0 renamed CRT_{A0}
- net MA1 renamed CRT_{A1}
- net MA10 renamed CRT_{A10}
- net MA11 renamed CRT_{A11}
- net CRT_{A11}: no longer U158.3 (I_{2})
- net MA12 renamed CRT_{A12}
- net CRT_{A12}: now also U158.3 (I_{2})
- net MA13 renamed CRT_{A13}
- net MA2 renamed CRT_{A2}
- net MA3 renamed CRT_{A3}
- net MA4 renamed CRT_{A4}
- net MA5 renamed CRT_{A5}
- net MA6 renamed CRT_{A6}
- net MA7 renamed CRT_{A7}
- net MA8 renamed CRT_{A8}
- net MA9 renamed CRT_{A9}
- net OSC renamed 14MHz
- net O_{1} renamed CLT_{O1}
- net SRAM_WR_TIMING renamed SRAM_{WE_STR}
- net U133_~{QA} renamed ~{U133_{QA}}
- net XA0 renamed CPU_{A0}
- net XA1 renamed CPU_{A1}
- net XA11 renamed CPU_{A11}
- net XA12 renamed CPU_{A12}
- net XA13 renamed CPU_{A13}
- net XA2 renamed CPU_{A2}
- net ~{CC_REG_{SEL}} renamed ~{CC_REG_{CS}}
- net ~{MODE_REG_{SEL}} renamed ~{MODE_REG_{CS}}
- net ~{MUX_IN_{A}} renamed CRM_{A13}
- net ~{OPTION_REG_1_{SEL}} renamed ~{OPTION_REG_1_{CS}}
- net ~{OPTION_REG_3_{SEL}} renamed ~{OPTION_REG_3_{CS}}
- net ~{PAL_{OE}} renamed ~{VM_{RD}}
- net ~{RESET} renamed ~{RESET_{BRD}}
- net ~{SRAM_{DECODE}} renamed ~{SRAM_{EN}}
- net ~{SRAM_{WE}} renamed ~{SRAM_{WR}}
- net ~{STATUS_REG_{SEL}} renamed ~{STATUS_REG_{CS}}
- net ~{VRAM_{DECODE_Q}} renamed VRAM_{DECODE_Q}
- new net CC_D0: U121.10 (E)
- new net CC_D1: U123.10 (E)
- new net CC_D2: U121.11 (F)
- new net CC_D3: U123.11 (F)
- new net CC_D4: U121.12 (G)
- new net CC_D5: U123.12 (G)
- new net CC_D6: U121.14 (H)
- new net CC_D7: U123.14 (H)
- no-connect marks 13 -> 28
Other:
- added sheet Main Registers (video_regs.kicad_sch)
- added sheet Palette Registers (palette_regs.kicad_sch)
- sheet Font SRAM ports: added CPU_{A[0..19]}, {X_BUS}, ~{SRAM_{EN}}, ~{SRAM_{RD}}, ~{SRAM_{WR}}; removed XA[0..19], ~{SRAM_{DECODE}}, ~{SRAM_{WE}}
- sheet Video RAM ports: added CPU_{A[0..19]}, CRM_{A12}, CRM_{A13}, CRT_{A[0..13]}, {X_BUS}, ~{VMUX_{CPU}}, ~{VMUX_{CRT}}, ~{VM_{RAS_T}}, ~{VM_{WR_T}}; removed MA[0..13], VA[0..7]
- note added: "To DCON (Page 9)"
- moved on the sheet: U107, U109, U111, U112A, U112B, U114, U116A, U116B, U117B, U117C, U117D, U117F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

Commit message: More updates
Parts:
- removed U109, U121, U123: 74LS166, Package_DIP:DIP-16_W7.62mm, symbol 74xx:74LS166
- removed U131: 74LS240, Package_DIP:DIP-20_W7.62mm, symbol 74xx:74LS240
- removed unit 1 of U132
- removed unit 2 of U133
- removed unit 1 of U133
- removed unit 4 of U139
- removed unit 2 of U139
- removed unit 1 of U139
- removed U151: PAL20L2, Package_DIP:DIP-24_W7.62mm, symbol seequa:PAL20L2
- added U163: 74LS00, Package_DIP:DIP-14_W7.62mm_Socket, symbol 74xx:74LS00
- U111: value PAL18L4CNS -> PAL18L4; seq_notes Character Color MUX -> Color MUX
Connections:
- net AT_D7: now also U155.1
- net BLINK_{EN}: now also U111.21 (I_{16}), U155.2
- net CRTC_{EN}: now also U134.9 (Q)
- net HSYNC_{EXT}: now also U138.13 (O6b)
- net VSYNC_{EXT}: now also U138.11 (O5b)
- net ~{CC_REG_{CS}}: no longer U126.14 (O1)
- net ~{MODE_REG_{CS}}: no longer U126.15 (O0)
- net ~{XIOW}: now also U163.1
- net ~{BLINK_ACTIVE}: now reaches U111.2 (I_{1}), U155.12
- net at U134.13 (~{R}): now also U163.3
- net I_{L}: now reaches U111.4 (I_{3}), U114.9 (O3)
- net R_{L}: now reaches U111.5 (I_{4}), U114.6 (O2)
- net G_{L}: now reaches U111.6 (I_{5}), U114.5 (O1)
- net B_{L}: now reaches U111.7 (I_{6}), U114.2 (O0)
- net Composite Generation/CMP_{b}: now reaches U135.5 (O1), U138.10 (I4)
- net ~{VSYNC_OUT}: now reaches U138.12 (I5), U139.8
- net Composite Generation/CMP_{r}: now reaches U135.9 (O3), U138.4 (I2)
- net Composite Generation/CMP_{g}: now reaches U135.6 (O2), U138.6 (I3)
- net CLT_{O1} renamed CLT_{O2}
- net PAL0 renamed CLUT0
- net PAL1 renamed CLUT1
- net PAL2 renamed CLUT2
- net PAL3 renamed CLUT3
- net PCLK renamed CLK_{88}
- net VRAM_{DECODE_Q} renamed VMEM_{DECODE_Q}
- net ~{CMX_{O0}_DLY} renamed ~{CMX_{b}}
- net ~{CMX_{O0}} renamed ~{CMX_{b}'}
- net ~{CMX_{O1}_DLY} renamed ~{CMX_{g}}
- net ~{CMX_{O1}} renamed ~{CMX_{g}'}
- net ~{CMX_{O2}_DLY} renamed ~{CMX_{i}}
- net ~{CMX_{O2}} renamed ~{CMX_{i}'}
- net ~{CMX_{O3}_DLY} renamed ~{CMX_{r}}
- net ~{CMX_{O3}} renamed ~{CMX_{r}'}
- new net Main Registers/~{CC_REG_{CS}}: U126.14 (O1)
- new net Main Registers/~{MODE_REG_{CS}}: U126.15 (O0)
- new net ~{XIOR}: U163.2
- no-connect marks 28 -> 27
Other:
- added sheet Serializers (video_serializers.kicad_sch)
- sheet Composite Generation ports: added 14MHz, BW, C0_{BODGE_IN}, CLT_{O2}, CMP_{b}, CMP_{g}, CMP_{r}, ~{14MHz}, ~{3.58MHz}; removed none
- sheet Font SRAM ports: added none; removed ~{SRAM1_{CE}}, ~{SRAM_{OE}}
- note added: "Attribute Byte"
- note added: "Palette Entry"
- moved on the sheet: J11, U107, U111, U112A, U112B, U114, U116A, U116B, U117B, U117C, U117D, U117F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

Commit message: Add parallel port, game port
Parts:
- removed U107: 74LS157, Package_DIP:DIP-16_W7.62mm, symbol 74xx:74LS157
- removed U111, U146: PAL18L4, Package_DIP:DIP-24_W7.62mm, symbol seequa:PAL18L4
- removed U114, U135: 74F374, Package_DIP:DIP-20_W7.62mm, symbol 74xx:74LS374
- removed unit 6 of U117
- removed U126: 74LS138, Package_DIP:DIP-16_W7.62mm, symbol 74xx:74LS138
- removed unit 2 of U134
- removed unit 1 of U134
- removed unit 2 of U136
- removed unit 3 of U136
- removed unit 3 of U139
- removed U154: 74LS161, Package_DIP:DIP-16_W7.62mm, symbol 74xx:74LS161
- removed unit 3 of U155
- removed unit 1 of U155
- removed U163: 74LS00, Package_DIP:DIP-14_W7.62mm_Socket, symbol 74xx:74LS00
- removed U58: HD46505SP, Package_DIP:DIP-40_W15.24mm, symbol GPU:MC6845
- removed U98: DMPAL12L6NC, Package_DIP:DIP-20_W7.62mm, symbol seequa:PAL12L6
- added C92: C_Bypass_Ceramic_2.54mm, seequa_footprints:C_Seequa_Bypass_2.54mm, symbol seequa:C_Bypass_Ceramic_2.54mm
Connections:
- net +5V: now also C92.1
- net GND: now also U138.15 (OEb), C92.2
- net HSYNC_{EXT}: now also J11.8 (Pin_8); no longer J11.9 (Pin_9)
- net VSYNC_{EXT}: now also J11.9 (Pin_9); no longer J11.8 (Pin_8)
- net ~{VM_{WR_T}}: now also U158.17 (I/~{O_{4}})
- net ~{VM_{WR}}: no longer U158.17 (I/~{O_{4}})
- net RASTER_{i}: now reaches U138.2 (I1)
- net Composite Generation/CMP_{b} renamed RASTER_{b}
- net Composite Generation/CMP_{g} renamed RASTER_{g}
- net Composite Generation/CMP_{r} renamed RASTER_{r}
- net ~{HSYNC} renamed Composite Generation/~{HSYNC}
- net ~{VSYNC_OUT} renamed Sync Timings/~{VSYNC_OUT}
- no-connect marks 27 -> 14
Other:
- added sheet Address Decoders (video_decoders.kicad_sch)
- added sheet CRTC (crtc.kicad_sch)
- added sheet Rasterization Pipeline (rasterization.kicad_sch)
- sheet Composite Generation ports: added CMP_{I}, CRTC_HS, CRTC_VS, GRAPHICS, HSYNC, VMEM_{EN}, VSYNC_OUT, ~{HSYNC}; removed none
- sheet Font SRAM ports: added 16MHz, {~{BUS_SIGNALS}}; removed ~{SRAM_{RD}}, ~{SRAM_{WR}}
- sheet Main Registers ports: added ~{STATUS_REG_{CS}}; removed ~{PALETTE0_{WR}}, ~{PALETTE1_{WR}}
- sheet Sync Timings ports: added FRONT_PORCH, HSYNC, VSYNC_OUT, ~{HSYNC}, ~{VSYNC_OUT}; removed none
- note added: "From NOVRAM Decoder (Page 4)"
- note added: "To CPU Logic (Page 2)"
- moved on the sheet: J11, U112A, U112B, U112C, U116A, U116B, U117B, U117C, U117D, U127E, U137, U138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

Commit message: Updates, chameleon logo
Other:
- sheet Address Decoders ports: added none; removed ~{VIDEO_DECODER_{EN}}
- sheet Palette Registers ports: added {CLUT}; removed CLUT[0..3]
- sheet Video RAM ports: added ~{VM_{RDGATE}}; removed none
Changed lines of the file:
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@@
 	)
 	(junction
-		(at 345.44 177.8)
+		(at 179.07 231.14)
 		(diameter 0)
 		(color 0 0 0 0)
 	)
 	(junction
-		(at 179.07 229.87)
+		(at 345.44 177.8)
 		(diameter 0)
-		(color 0 0 0 1)
+		(color 0 0 0 0)
 	)
 	(junction
@@
 		)
 	)
+	(wire
+		(pts
+			(xy 179.07 231.14) (xy 179.07 233.68)
+		)
+		(stroke
+			(width 0.25)
+			(type default)
+			(color 0 0 0 1)
+		)
+	)
 	(bus
 		(pts
@@
 	(wire
 		(pts
-			(xy 71.12 25.4) (xy 72.39 25.4)
-		)
-		(stroke
-			(width 0)
-			(type default)
-		)
-	)
-	(wire
-		(pts
 			(xy 508 274.32) (xy 549.91 274.32)
 		)
@@
 		)
 	)
-	(wire
-		(pts
-			(xy 179.07 229.87) (xy 179.07 233.68)
-		)
-		(stroke
-			(width 0.25)
-			(type default)
-			(color 0 0 0 1)
-		)
-	)
 	(bus
 		(pts
@@
 	(wire
 		(pts
-			(xy 71.12 19.05) (xy 71.12 25.4)
+			(xy 143.51 95.25) (xy 158.75 95.25)
 		)
 		(stroke
@@
 	(wire
 		(pts
-			(xy 36.83 19.05) (xy 71.12 19.05)
-		)
-		(stroke
-			(width 0)
-			(type default)
-		)
-	)
-	(wire
-		(pts
 			(xy 92.71 77.47) (xy 132.08 77.47)
 		)
@@
 	(wire
 		(pts
-			(xy 15.24 229.87) (xy 15.24 570.23)
+			(xy 15.24 231.14) (xy 15.24 570.23)
 		)
 		(stroke
@@
 	(wire
 		(pts
-			(xy 15.24 229.87) (xy 179.07 229.87)
+			(xy 15.24 231.14) (xy 179.07 231.14)
 		)
 		(stroke
@@
 	(wire
 		(pts
-			(xy 179.07 220.98) (xy 179.07 229.87)
+			(xy 179.07 220.98) (xy 179.07 231.14)
 		)
 		(stroke
@@
 		)
 	)
+	(label "~{VM_{RDGATE}}"
+		(at 143.51 95.25 0)
+		(effects
+			(font
+				(size 1.27 1.27)
+			)
+			(justify left bottom)
+		)
+	)
 	(label "~{VM_{CAS}}"
 		(at 613.41 198.12 180)
@@
 		)
 	)
-	(label "CLUT[0..3]"
-		(at 344.17 107.95 0)
-		(effects
-			(font
-				(size 1.27 1.27)
-			)
-			(justify left bottom)
-		)
-	)
 	(label "~{VM_{CAS_T}}"
 		(at 224.79 104.14 180)
@@
 		)
 	)
-	(global_label "~{VIDEO_DECODER_{EN}}"
-		(shape input)
-		(at 36.83 19.05 180)
-		(fields_autoplaced yes)
-		(effects
-			(font
-				(size 1.27 1.27)
-			)
-			(justify right)
-		)
-		(property "Intersheetrefs" "${INTERSHEET_REFS}"
-			(at 16.6914 19.05 0)
-			(effects
-				(font
-					(size 1.27 1.27)
-				)
-				(justify right)
-				(hide yes)
-			)
-		)
-	)
 	(hierarchical_label "PD[0..7]"
 		(shape bidirectional)
@@
 		)
 		(pin "~{VM_{RD}}" input
-			(at 132.08 44.45 0)
+			(at 132.08 46.99 0)
 			(effects
 				(font
@@
 			)
 		)
-		(pin "~{VIDEO_DECODER_{EN}}" input
-			(at 72.39 25.4 180)
-			(effects
-				(font
-					(size 1.27 1.27)
-				)
-				(justify left)
-			)
-		)
 		(pin "~{CC_REG_{CS}}" input
 			(at 132.08 38.1 0)
@@
 			)
 		)
+		(pin "~{VM_{RDGATE}}" input
+			(at 158.75 95.25 180)
+			(effects
+				(font
+					(size 1.27 1.27)
+				)
+				(justify left)
+			)
+		)
 		(instances
 			(project "seequa_chameleon"
@@
 			)
 		)
-		(pin "CLUT[0..3]" input
-			(at 314.96 107.95 0)
-			(effects
-				(font
-					(size 1.27 1.27)
-				)
-				(justify right)
-			)
-		)
 		(pin "PD[0..7]" input
 			(at 265.43 110.49 180)
@@
 			)
 		)
+		(pin "{CLUT}" input
+			(at 314.96 107.95 0)
+			(effects
+				(font
+					(size 1.27 1.27)
+				)
+				(justify right)
+			)
+		)
