File: kicad/video_clock.kicad_sch (KiCad schematic)
At the start: 6 parts, among them U136 74LS04, X2 14.31818MHz

Commit message: update kicad project
Parts:
- added TP1: TestPoint, TestPoint:TestPoint_Pad_D1.5mm, symbol Connector:TestPoint
- C90: seq_coord (none) -> E23
- C91: seq_coord (none) -> F23
- R42: seq_coord (none) -> E23; seq_silkscreen R1 -> (none)
- R43: seq_coord (none) -> E23; seq_silkscreen R2 -> (none)
- U136: seq_coord (none) -> F23; seq_silkscreen (none) -> LS04
- X2: seq_coord (none) -> E22
Connections:
- net ~{14.31818MHz}: now also TP1.1
Changed lines of the file:
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@@
+	)
+	(junction
+		(at 194.31 83.82)
+		(diameter 0)
+		(color 0 0 0 0)
 	)
 	(junction
@@
 	(wire
 		(pts
-			(xy 190.5 83.82) (xy 198.12 83.82)
+			(xy 190.5 83.82) (xy 194.31 83.82)
 		)
 		(stroke
@@
 	(wire
 		(pts
+			(xy 194.31 83.82) (xy 198.12 83.82)
+		)
+		(stroke
+			(width 0)
+			(type default)
+		)
+	)
+	(wire
+		(pts
 			(xy 175.26 83.82) (xy 175.26 93.98)
+		)
+		(stroke
+			(width 0)
+			(type default)
+		)
+	)
+	(wire
+		(pts
+			(xy 194.31 77.47) (xy 194.31 83.82)
 		)
 		(stroke
@@
 			)
 		)
-		(property "seq_coord" ""
+		(property "seq_coord" "E23"
 			(at 127 109.22 0)
 			(effects
@@
 			)
 		)
-		(property "seq_coord" ""
+		(property "seq_coord" "F23"
 			(at 182.88 83.82 0)
 			(effects
@@
 			)
 		)
-		(property "seq_silkscreen" ""
+		(property "seq_silkscreen" "LS04"
 			(at 182.88 83.82 0)
 			(effects
@@
 					(reference "U136")
 					(unit 6)
+				)
+			)
+		)
+	)
+	(symbol
+		(lib_id "Connector:TestPoint")
+		(at 194.31 77.47 0)
+		(unit 1)
+		(exclude_from_sim no)
+		(in_bom yes)
+		(on_board yes)
+		(dnp no)
+		(fields_autoplaced yes)
+		(property "Reference" "TP1"
+			(at 196.85 72.8979 0)
+			(effects
+				(font
+					(size 1.27 1.27)
+				)
+				(justify left)
+			)
+		)
+		(property "Value" "TestPoint"
+			(at 196.85 75.4379 0)
+			(effects
+				(font
+					(size 1.27 1.27)
+				)
+				(justify left)
+			)
+		)
+		(property "Footprint" "TestPoint:TestPoint_Pad_D1.5mm"
+			(at 199.39 77.47 0)
+			(effects
+				(font
+					(size 1.27 1.27)
+				)
+				(hide yes)
+			)
+		)
+		(property "Datasheet" "~"
+			(at 199.39 77.47 0)
+			(effects
+				(font
+					(size 1.27 1.27)
+				)
+				(hide yes)
+			)
+		)
+		(property "Description" "test point"
+			(at 194.31 77.47 0)
+			(effects
+				(font
+					(size 1.27 1.27)
+				)
+				(hide yes)
+			)
+		)
+		(property "seq_partno" ""
+			(at 194.31 77.47 0)
+			(effects
+				(font
+					(size 1.27 1.27)
+				)
+				(hide yes)
+			)
+		)
+		(property "seq_coord" ""
+			(at 194.31 77.47 0)
+			(effects
+				(font
+					(size 1.27 1.27)
+				)
+				(hide yes)
+			)
+		)
+		(property "seq_silkscreen" ""
+			(at 194.31 77.47 0)
+			(effects
+				(font
+					(size 1.27 1.27)
+				)
+				(hide yes)
+			)
+		)
+		(property "seq_sharpie" ""
+			(at 194.31 77.47 0)
+			(effects
+				(font
+					(size 1.27 1.27)
+				)
+				(hide yes)
+			)
+		)
+		(property "seq_notes" ""
+			(at 194.31 77.47 0)
+			(effects
+				(font
+					(size 1.27 1.27)
+				)
+				(hide yes)
+			)
+		)
+		(property "seq_port" ""
+			(at 194.31 77.47 0)
+			(effects
+				(font
+					(size 1.27 1.27)
+				)
+				(hide yes)
+			)
+		)
+		(pin "1"
+		)
+		(instances
+			(project ""
+				(path "/ae890d4c-6a02-4621-80ce-7ef4317218ea/a308f48d-1c03-4054-a3cd-412839ec499d/77e51b0e-bae8-416e-b9d8-861e4af44b64"
+					(reference "TP1")
+					(unit 1)
 				)
 			)
@@
 			)
 		)
-		(property "seq_coord" ""
+		(property "seq_coord" "F23"
 			(at 165.1 83.82 0)
 			(effects
@@
 			)
 		)
-		(property "seq_silkscreen" ""
+		(property "seq_silkscreen" "LS04"
 			(at 165.1 83.82 0)
 			(effects
@@
 			)
 		)
-		(property "seq_coord" ""
+		(property "seq_coord" "F23"
 			(at 139.7 83.82 0)
 			(effects
@@
 			)
 		)
-		(property "seq_silkscreen" ""
+		(property "seq_silkscreen" "LS04"
 			(at 139.7 83.82 0)
 			(effects
@@
 			)
 		)
-		(property "seq_coord" ""
+		(property "seq_coord" "F23"
 			(at 133.35 99.06 0)
 			(effects
@@
 			)
 		)
-		(property "seq_coord" ""
+		(property "seq_coord" "E23"
 			(at 139.7 68.58 0)
 			(effects
@@
 			)
 		)
-		(property "seq_silkscreen" "R1"
+		(property "seq_silkscreen" ""
 			(at 139.7 68.58 0)
 			(effects
@@
 			)
 		)
-		(property "seq_coord" ""
+		(property "seq_coord" "E23"
 			(at 163.83 93.98 0)
 			(effects
@@
 			)
 		)
-		(property "seq_silkscreen" "R2"
+		(property "seq_silkscreen" ""
 			(at 163.83 93.98 0)
 			(effects
@@
 			)
 		)
-		(property "seq_coord" ""
+		(property "seq_coord" "E22"
 			(at 143.51 99.06 0)
 			(effects
