File: kicad/video_decoders.kicad_sch (KiCad schematic)
At the start: 2 parts, among them U126 74LS138, U98 DMPAL12L6NC

Commit message: Updates, chameleon logo
Changed lines of the file:
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@@
+	)
+	(junction
+		(at 53.34 62.23)
+		(diameter 0)
+		(color 0 0 0 0)
 	)
 	(junction
@@
 	)
 	(bus_entry
+		(at 139.7 93.98)
+		(size 2.54 2.54)
+		(stroke
+			(width 0)
+			(type default)
+		)
+	)
+	(bus_entry
 		(at 67.31 78.74)
 		(size 2.54 2.54)
@@
 		)
 	)
+	(bus
+		(pts
+			(xy 139.7 62.23) (xy 139.7 93.98)
+		)
+		(stroke
+			(width 0.75)
+			(type default)
+			(color 194 194 0 1)
+		)
+	)
 	(wire
 		(pts
@@
 		)
 	)
+	(bus
+		(pts
+			(xy 53.34 62.23) (xy 139.7 62.23)
+		)
+		(stroke
+			(width 0.75)
+			(type default)
+			(color 194 194 0 1)
+		)
+	)
 	(wire
 		(pts
@@
 		)
 	)
+	(wire
+		(pts
+			(xy 142.24 96.52) (xy 163.83 96.52)
+		)
+		(stroke
+			(width 0)
+			(type default)
+		)
+	)
 	(bus
 		(pts
@@
 			(type default)
 			(color 204 102 0 1)
-		)
-	)
-	(wire
-		(pts
-			(xy 157.48 96.52) (xy 163.83 96.52)
-		)
-		(stroke
-			(width 0)
-			(type default)
 		)
 	)
@@
 	(label "XA18"
 		(at 71.12 96.52 0)
+		(effects
+			(font
+				(size 1.27 1.27)
+			)
+			(justify left bottom)
+		)
+	)
+	(label "~{VIDEO_DECODER_{EN}}"
+		(at 144.78 96.52 0)
 		(effects
 			(font
@@
 		)
 	)
-	(hierarchical_label "~{VIDEO_DECODER_{EN}}"
-		(shape input)
-		(at 157.48 96.52 180)
-		(effects
-			(font
-				(size 1.27 1.27)
-			)
-			(justify right)
-		)
-	)
